File: hardware/midicade.kicad_pcb (KiCad board)
At the start: 2 copper layers, 140 x 140 mm, 65 parts, among them J1 Conn_01x02, J10 Conn_01x02, J11 Conn_01x02, J12 Conn_01x02, J13 Conn_01x02, J14 Conn_01x02, J15 Conn_01x02, J16 Conn_01x02, J17 USB_B, J18 Conn_01x06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

Commit message: minor production changes
Parts:
- removed D1: 1N4148, Diode_SMD:D_SOD-323
- added REF**: KiCad-Logo2_6mm_SilkScreen, Symbol:KiCad-Logo2_6mm_SilkScreen, F.Cu at (90.0, 121.0)
- moved C4 6.00 mm to (69.0, 37.8)
- moved R4 6.00 mm to (72.0, 37.8)
- moved R5 6.00 mm to (66.0, 37.8)
- turned SW1 to 270 degrees
Routing:
- net /RESET: track 62.5 -> 53.1 mm
- net +5V: track 457.7 -> 452.0 mm
- net Net-(R5-Pad2): track 8.34 -> 7.07 mm
- net GND: track 154.2 -> 154.7 mm

Commit message: rev 1.2 hardware
Parts:
- removed R5: 330, Resistor_SMD:R_0603_1608Metric
- removed REF**: KiCad-Logo2_6mm_SilkScreen, Symbol:KiCad-Logo2_6mm_SilkScreen
- removed SW1: SW_Push, Resources:SW_SPST_Omron_B3FS-100xP_3D
- R4: value 4.7K -> 10K
- R7: value 1K -> 470
Connections:
- net /D16 renamed /D20
- net /D17 renamed /D21
- J1 pad 1: /D18 -> /D22
- J10 pad 1: /D15 -> /D19
- J2 pad 1: /D19 -> /D23
- J6 pad 1: /D14 -> /D18
- U1 pad 36: /D14 -> /D18
- U1 pad 37: /D15 -> /D19
- U1 pad 40: /D18 -> /D22
- U1 pad 41: /D19 -> /D23
Routing:
- net /D15: track 19.0 -> 0.00 mm
- net /D22: track 0.00 -> 18.7 mm
- net /D14: track 10.7 -> 0.00 mm
- net /D23: track 0.00 -> 10.4 mm
- net /D19: track 10.4 -> 19.0 mm
- net /D18: track 18.7 -> 10.7 mm
- net Net-(R5-Pad2): track 7.07 -> 0.00 mm
- net GND: track 154.7 -> 148.4 mm
- net /RESET: track 53.1 -> 50.1 mm
- net /DN: track 32.5 -> 33.3 mm
Other:
- board text added: "Rev 1.2 github.com/tapir/midicade"
- board text removed: "Rev 1.0 github.com/tapir/midicade"
